File: qt45.kicad_pcb (KiCad board)
At the start: 2 copper layers, 106 parts, among them SW1 SW_PUSH, U1 ATmega32U4-AU, Y1 16MHz

Commit message: Rough placement of components
Parts:
- C1, C2, C3, C4, C5, C6, C7, F1, R1, R2, R3, R4, U1, USB1, Y1: moved to B.Cu
- MX23: footprint MX_Alps_Hybrid:MXOnly-6.25U-NoLED -> MX_Alps_Hybrid:MXOnly-6.25U-ReversedStabilizers-NoLED
- moved U1 211.0 mm to (171.1, 123.8), turned to 270 degrees
- moved SW1 202.9 mm to (128.0, 123.3)
- moved C1 183.1 mm to (182.9, 128.1)
- moved C2 172.4 mm to (182.9, 119.3), turned to 180 degrees
- moved C4 169.5 mm to (174.6, 133.0)
- moved C3 160.1 mm to (162.1, 127.5), turned to 90 degrees
- moved R4 159.5 mm to (168.0, 133.0), turned to 180 degrees
- moved C5 153.9 mm to (176.1, 114.8)
- moved C6 146.3 mm to (162.1, 120.3), turned to 270 degrees
- moved Y1 145.1 mm to (182.9, 123.7), turned to 90 degrees
- moved R3 139.1 mm to (128.1, 119.4), turned to 180 degrees
- moved USB1 138.8 mm to (146.1, 43.7), turned to 270 degrees
- moved C7 134.9 mm to (170.7, 114.8), turned to 180 degrees
- moved R1 78.2 mm to (144.5, 53.1), turned to 270 degrees
- moved R2 63.2 mm to (146.8, 53.1), turned to 270 degrees
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
Commit message: Route key switches
Parts:
- moved D20 15.9 mm to (128.6, 71.4)
- moved D29 15.9 mm to (161.9, 109.5)
- moved D43 15.9 mm to (261.9, 71.4)
- moved D45 15.9 mm to (261.9, 109.5)
- turned R1 to 90 degrees
- turned R2 to 90 degrees
Routing:
- net ROW1: track 0.00 -> 238.1 mm
- net ROW0: track 0.00 -> 231.8 mm
- net ROW2: track 0.00 -> 224.6 mm
- net COL6: track 0.00 -> 68.0 mm
- net COL11: track 0.00 -> 67.0 mm
- net COL10: track 0.00 -> 66.0 mm
- net COL2: track 0.00 -> 65.0 mm
- net COL3: track 0.00 -> 64.1 mm
- net COL7: track 0.00 -> 44.0 mm
- net COL13: track 0.00 -> 44.0 mm
- net COL9: track 0.00 -> 44.0 mm
- net COL4: track 0.00 -> 44.0 mm
- net COL5: track 0.00 -> 44.0 mm
- net COL8: track 0.00 -> 44.0 mm
- net ROW3: track 0.00 -> 42.9 mm
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Other:
- board outline added: 266.7 x 76.2 mm
- net class Default: trace_width 0.25 -> 0.254
- net class Power added: clearance 0.2, trace_width 0.381, via_dia 0.8, via_drill 0.4

Commit message: Routing (no rows and columns)
Parts:
- moved R3 35.3 mm to (161.2, 131.8), turned to 270 degrees
- moved R4 31.4 mm to (199.1, 137.2)
- moved R2 28.5 mm to (152.3, 81.1)
- moved R1 28.4 mm to (149.5, 81.1)
- moved F1 27.8 mm to (146.4, 80.0)
- moved USB1 26.5 mm to (148.4, 70.0)
- moved C4 24.5 mm to (199.1, 133.9)
- moved D21 17.5 mm to (135.8, 101.6)
- moved C5 12.6 mm to (182.0, 125.9)
- moved C6 11.8 mm to (164.5, 131.8)
- moved C2 11.8 mm to (185.3, 130.8)
- moved C7 11.5 mm to (173.5, 125.9), turned to 90 degrees
- moved D22 11.4 mm to (142.1, 120.7)
- moved D39 11.4 mm to (237.3, 120.7)
- moved D45 11.4 mm to (264.3, 120.7)
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Connections:
- D36 pad 1: ROW3 -> ROW4
- D40 pad 1: ROW3 -> ROW4
Routing:
- net GND: track 0.00 -> 391.7 mm, vias 0 -> 1
- net +5V: track 0.00 -> 179.6 mm, vias 0 -> 6
- net Net-(R3-Pad2): track 0.00 -> 70.6 mm, vias 0 -> 3
- net Net-(R1-Pad1): track 0.00 -> 69.9 mm, vias 0 -> 2
- net Net-(R2-Pad1): track 0.00 -> 69.2 mm, vias 0 -> 2
- net ROW3: track 42.9 -> 95.6 mm
- net Net-(R4-Pad2): track 0.00 -> 32.8 mm
- net ROW4: track 0.00 -> 21.4 mm
- net Net-(D43-Pad2): track 0.00 -> 16.0 mm
- net Net-(C2-Pad1): track 0.00 -> 11.1 mm
- net Net-(D23-Pad2): track 0.00 -> 10.4 mm
- net Net-(C1-Pad1): track 0.00 -> 8.47 mm
- net D+: track 0.00 -> 7.20 mm
- net D-: track 0.00 -> 6.38 mm
- net Net-(D21-Pad2): track 10.4 -> 16.0 mm
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
Commit message: Routing fixes
Parts:
- turned SW1 to 180 degrees
Routing:
- net GND: track 391.7 -> 401.8 mm
- net +5V: track 179.6 -> 185.3 mm, vias 6 -> 7
- net Net-(R3-Pad2): track 70.6 -> 67.6 mm
- net Net-(U1-Pad32): track 0.00 -> 0.78 mm

Commit message: Start reroute
Parts:
- moved C1 78.8 mm to (106.8, 130.7), turned to 180 degrees
- moved C2 78.8 mm to (106.8, 138.6), turned to 0 degrees
- moved Y1 78.4 mm to (106.8, 134.6), turned to 270 degrees
- moved C5 72.0 mm to (111.5, 140.6), turned to 180 degrees
- moved C4 71.2 mm to (128.3, 140.6)
- moved U1 53.6 mm to (119.9, 134.9), turned to 90 degrees
- moved C3 50.3 mm to (115.7, 126.2), turned to 180 degrees
- moved SW1 46.3 mm to (176.7, 134.4)
- moved C7 43.3 mm to (132.7, 140.6), turned to 0 degrees
- moved C6 34.4 mm to (130.2, 129.0), turned to 0 degrees
- moved D22 16.1 mm to (126.2, 118.3)
- moved F1 5.82 mm to (146.8, 85.8)
- moved R1 4.70 mm to (149.5, 85.8)
- moved R2 4.70 mm to (152.3, 85.8)
- moved D12 2.38 mm to (84.9, 118.3)
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Connections:
- MX23 pad 1: COL6 -> COL7
Routing:
- net GND: track 401.8 -> 63.1 mm, vias 1 -> 0
- net +5V: track 185.3 -> 110.8 mm, vias 7 -> 8
- net ROW3: track 95.6 -> 21.4 mm
- net Net-(R3-Pad2): track 67.6 -> 0.00 mm, vias 3 -> 0
- net ROW2: track 224.6 -> 189.7 mm
- net ROW1: track 238.1 -> 203.2 mm
- net Net-(R4-Pad2): track 32.8 -> 0.00 mm
- net COL6: track 68.0 -> 44.0 mm
- net COL7: track 44.0 -> 66.0 mm
- net Net-(D23-Pad2): track 10.4 -> 0.00 mm
- net D+: track 7.20 -> 12.9 mm, vias 0 -> 2
- net VCC: track 4.24 -> 9.90 mm, vias 0 -> 2
- net D-: track 6.38 -> 11.1 mm, vias 0 -> 2
- net Net-(R2-Pad1): track 69.2 -> 73.8 mm
- net Net-(D22-Pad2): track 10.4 -> 13.6 mm
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
Commit message: More routing
Parts:
- moved R4 69.9 mm to (130.2, 125.7)
- moved R3 65.2 mm to (96.0, 134.4), turned to 0 degrees
- moved C7 36.8 mm to (96.0, 137.7), turned to 180 degrees
- moved USB1 4.76 mm to (148.4, 65.3)
- moved C4 3.17 mm to (130.2, 138.0)
- moved C3 0.51 mm to (115.7, 125.7)
Connections:
- D23 pad 1: ROW3 -> ROW4
- U1 pad 18: Net-(U1-Pad18) -> ROW3
- U1 pad 19: Net-(U1-Pad19) -> ROW0
- U1 pad 20: Net-(U1-Pad20) -> ROW1
- U1 pad 21: Net-(U1-Pad21) -> ROW2
- U1 pad 22: Net-(U1-Pad22) -> COL5
- U1 pad 27: Net-(U1-Pad27) -> COL6
- U1 pad 28: Net-(U1-Pad28) -> COL4
- U1 pad 29: Net-(U1-Pad29) -> COL3
- U1 pad 30: Net-(U1-Pad30) -> COL2
- U1 pad 31: Net-(U1-Pad31) -> COL0
- U1 pad 32: Net-(U1-Pad32) -> COL1
Routing:
- net COL0: track 41.1 -> 198.8 mm
- net GND: track 63.1 -> 209.2 mm, vias 0 -> 1
- net COL1: track 21.0 -> 162.0 mm
- net ROW0: track 231.8 -> 366.2 mm, vias 0 -> 2
- net COL2: track 65.0 -> 194.9 mm
- net ROW1: track 203.2 -> 318.1 mm, vias 0 -> 2
- net COL3: track 64.1 -> 174.2 mm
- net Net-(R3-Pad2): track 0.00 -> 106.5 mm, vias 0 -> 1
- net COL4: track 44.0 -> 134.7 mm
- net ROW4: track 21.4 -> 92.9 mm
- net COL6: track 44.0 -> 84.6 mm
- net ROW3: track 21.4 -> 58.7 mm
- net Net-(C7-Pad1): track 0.00 -> 28.7 mm
- net COL5: track 44.0 -> 63.1 mm, vias 0 -> 1
- net ROW2: track 189.7 -> 207.5 mm
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Other:
- board size 266.7 x 76.2 mm -> 266.7 x 81 mm

Commit message: First draft of routing
Parts:
- moved C4 2.54 mm to (130.2, 140.6)
Connections:
- D23 pad 1: ROW4 -> ROW3
- D36 pad 1: ROW4 -> ROW3
- D40 pad 1: ROW4 -> ROW3
- U1 pad 1: Net-(U1-Pad1) -> COL11
- U1 pad 25: Net-(U1-Pad25) -> COL6
- U1 pad 26: Net-(U1-Pad26) -> COL4
- U1 pad 27: COL6 -> COL3
- U1 pad 28: COL4 -> COL2
- U1 pad 29: COL3 -> COL0
- U1 pad 30: COL2 -> COL1
- U1 pad 31: COL0 -> Net-(U1-Pad31)
- U1 pad 32: COL1 -> Net-(U1-Pad32)
- U1 pad 36: Net-(U1-Pad36) -> COL8
- U1 pad 37: Net-(U1-Pad37) -> COL9
- U1 pad 38: Net-(U1-Pad38) -> COL10
- U1 pad 39: Net-(U1-Pad39) -> COL12
- U1 pad 40: Net-(U1-Pad40) -> COL13
- U1 pad 41: Net-(U1-Pad41) -> COL7
Routing:
- net ROW3: track 58.7 -> 221.1 mm, vias 0 -> 2
- net COL13: track 44.0 -> 199.4 mm, vias 0 -> 1
- net COL12: track 39.1 -> 172.7 mm, vias 0 -> 1
- net COL11: track 67.0 -> 182.6 mm, vias 0 -> 2
- net ROW4: track 92.9 -> 0.00 mm
- net COL10: track 66.0 -> 155.6 mm, vias 0 -> 2
- net COL9: track 44.0 -> 114.2 mm, vias 0 -> 1
- net COL8: track 44.0 -> 94.8 mm, vias 0 -> 1
- net ROW2: track 207.5 -> 242.6 mm, vias 0 -> 2
- net ROW1: track 318.1 -> 353.1 mm, vias 2 -> 4
- net +5V: track 126.0 -> 146.3 mm, vias 7 -> 8
- net COL7: track 66.0 -> 84.4 mm, vias 0 -> 3
- net Net-(R1-Pad1): track 58.7 -> 76.5 mm, vias 1 -> 2
- net Net-(R2-Pad1): track 61.2 -> 78.9 mm, vias 1 -> 2
- net GND: track 209.2 -> 217.9 mm
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
Commit message: Add ground plane
Parts:
- moved F1 2.76 mm to (146.8, 83.1)
Routing:
- net VCC: track 14.7 -> 11.9 mm
- net +5V: track 146.3 -> 149.0 mm
- added copper zone on B.Cu, net GND
Changed lines of the file:
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@@
     (thickness 1.6)
     (drawings 14)
-    (tracks 623)
+    (tracks 618)
     (zones 0)
     (modules 106)
@@
     (add_net VCC)
   )
+  (module MX_Alps_Hybrid:MXOnly-1U-NoLED (layer F.Cu)
+    (at 138.90625 77.7875)
+    (fp_text reference MX20 (at 0 3.175) (layer Dwgs.User)
+      (effects (font (size 1 1) (thickness 0.15)))
+    )
+    (fp_text value MX-1U (at 0 -7.9375) (layer Dwgs.User)
+      (effects (font (size 1 1) (thickness 0.15)))
+    )
+    (fp_line (start -9.525 9.525) (end -9.525 -9.525) (layer Dwgs.User) (width 0.15))
+    (fp_line (start 9.525 9.525) (end -9.525 9.525) (layer Dwgs.User) (width 0.15))
+    (fp_line (start 9.525 -9.525) (end 9.525 9.525) (layer Dwgs.User) (width 0.15))
+    (fp_line (start -9.525 -9.525) (end 9.525 -9.525) (layer Dwgs.User) (width 0.15))
+    (fp_line (start -7 -7) (end -7 -5) (layer Dwgs.User) (width 0.15))
+    (fp_line (start -5 -7) (end -7 -7) (layer Dwgs.User) (width 0.15))
+    (fp_line (start -7 7) (end -5 7) (layer Dwgs.User) (width 0.15))
+    (fp_line (start -7 5) (end -7 7) (layer Dwgs.User) (width 0.15))
+    (fp_line (start 7 7) (end 7 5) (layer Dwgs.User) (width 0.15))
+    (fp_line (start 5 7) (end 7 7) (layer Dwgs.User) (width 0.15))
+    (fp_line (start 7 -7) (end 7 -5) (layer Dwgs.User) (width 0.15))
+    (fp_line (start 5 -7) (end 7 -7) (layer Dwgs.User) (width 0.15))
+    (pad "" np_thru_hole circle (at 5.08 0 48.0996) (size 1.75 1.75) (drill 1.75) (layers *.Cu *.Mask))
+    (pad "" np_thru_hole circle (at -5.08 0 48.0996) (size 1.75 1.75) (drill 1.75) (layers *.Cu *.Mask))
+    (pad 1 thru_hole circle (at -3.81 -2.54) (size 2.25 2.25) (drill 1.47) (layers *.Cu B.Mask)
+      (net 62 COL6))
+    (pad "" np_thru_hole circle (at 0 0) (size 3.9878 3.9878) (drill 3.9878) (layers *.Cu *.Mask))
+    (pad 2 thru_hole circle (at 2.54 -5.08) (size 2.25 2.25) (drill 1.47) (layers *.Cu B.Mask)
+      (net 29 "Net-(D20-Pad2)"))
+  )
   (module MX_Alps_Hybrid:MXOnly-6.25U-ReversedStabilizers-NoLED (layer F.Cu)
     (at 146.05 134.9375)
@@
   )
   (module MX_Alps_Hybrid:MXOnly-1U-NoLED (layer F.Cu)
-    (at 138.90625 77.7875)
-    (fp_text reference MX20 (at 0 3.175) (layer Dwgs.User)
-      (effects (font (size 1 1) (thickness 0.15)))
-    )
-    (fp_text value MX-1U (at 0 -7.9375) (layer Dwgs.User)
-      (effects (font (size 1 1) (thickness 0.15)))
-    )
-    (fp_line (start -9.525 9.525) (end -9.525 -9.525) (layer Dwgs.User) (width 0.15))
-    (fp_line (start 9.525 9.525) (end -9.525 9.525) (layer Dwgs.User) (width 0.15))
-    (fp_line (start 9.525 -9.525) (end 9.525 9.525) (layer Dwgs.User) (width 0.15))
-    (fp_line (start -9.525 -9.525) (end 9.525 -9.525) (layer Dwgs.User) (width 0.15))
-    (fp_line (start -7 -7) (end -7 -5) (layer Dwgs.User) (width 0.15))
-    (fp_line (start -5 -7) (end -7 -7) (layer Dwgs.User) (width 0.15))
-    (fp_line (start -7 7) (end -5 7) (layer Dwgs.User) (width 0.15))
-    (fp_line (start -7 5) (end -7 7) (layer Dwgs.User) (width 0.15))
-    (fp_line (start 7 7) (end 7 5) (layer Dwgs.User) (width 0.15))
-    (fp_line (start 5 7) (end 7 7) (layer Dwgs.User) (width 0.15))
-    (fp_line (start 7 -7) (end 7 -5) (layer Dwgs.User) (width 0.15))
-    (fp_line (start 5 -7) (end 7 -7) (layer Dwgs.User) (width 0.15))
-    (pad "" np_thru_hole circle (at 5.08 0 48.0996) (size 1.75 1.75) (drill 1.75) (layers *.Cu *.Mask))
-    (pad "" np_thru_hole circle (at -5.08 0 48.0996) (size 1.75 1.75) (drill 1.75) (layers *.Cu *.Mask))
-    (pad 1 thru_hole circle (at -3.81 -2.54) (size 2.25 2.25) (drill 1.47) (layers *.Cu B.Mask)
-      (net 62 COL6))
-    (pad "" np_thru_hole circle (at 0 0) (size 3.9878 3.9878) (drill 3.9878) (layers *.Cu *.Mask))
-    (pad 2 thru_hole circle (at 2.54 -5.08) (size 2.25 2.25) (drill 1.47) (layers *.Cu B.Mask)
-      (net 29 "Net-(D20-Pad2)"))
-  )
-  (module MX_Alps_Hybrid:MXOnly-1U-NoLED (layer F.Cu)
     (at 272.25625 77.7875)
     (fp_text reference MX43 (at 0 3.175) (layer Dwgs.User)
@@
   )
   (module Fuse:Fuse_1206_3216Metric (layer B.Cu)
-    (at 146.84375 85.82025 90)
+    (at 146.84375 83.058 90)
     (descr "Fuse SMD 1206 (3216 Metric), square (rectangular) end terminal, IPC_7351 nominal, (Body size source: http://www.tortai-tech.com/upload/download/2011102023233369053.pdf), generated with kicad-footprint-generator")
     (tags resistor)
@@
   (segment (start 95.0745 134.366) (end 96.4715 132.969) (width 0.381) (layer B.Cu) (net 4))
   (segment (start 129.286 127.635) (end 129.286 128.9835) (width 0.381) (layer B.Cu) (net 4))
-  (segment (start 146.84375 87.22025) (end 146.84375 88.99525) (width 0.381) (layer B.Cu) (net 4))
-  (segment (start 146.84375 88.99525) (end 146.812 89.027) (width 0.381) (layer B.Cu) (net 4))
   (segment (start 129.413 127.635) (end 129.286 127.635) (width 0.381) (layer F.Cu) (net 4))
   (segment (start 129.286 128.9835) (end 129.2375 129.032) (width 0.381) (layer B.Cu) (net 4))
@@
   (segment (start 143.213311 107.865689) (end 143.213311 119.935893) (width 0.381) (layer B.Cu) (net 4))
   (segment (start 150.622 100.457) (end 143.213311 107.865689) (width 0.381) (layer B.Cu) (net 4))
-  (segment (start 146.84375 88.99525) (end 150.622 92.7735) (width 0.381) (layer B.Cu) (net 4))
-  (segment (start 150.622 92.7735) (end 150.622 100.457) (width 0.381) (layer B.Cu) (net 4))
   (segment (start 125.588 139.53) (end 125.588 138.874) (width 0.381) (layer B.Cu) (net 4))
   (segment (start 126.647 140.589) (end 125.588 139.53) (width 0.381) (layer B.Cu) (net 4))
@@
   (segment (start 116.6345 124.9195) (end 117.348 124.206) (width 0.381) (layer B.Cu) (net 4))
   (segment (start 117.348 124.206) (end 120.904 124.206) (width 0.381) (layer F.Cu) (net 4))
+  (segment (start 150.622 89.46598) (end 150.622 100.457) (width 0.381) (layer B.Cu) (net 4))
+  (segment (start 146.84375 85.68773) (end 150.622 89.46598) (width 0.381) (layer B.Cu) (net 4))
+  (segment (start 146.84375 84.458) (end 146.84375 85.68773) (width 0.381) (layer B.Cu) (net 4))
   (segment (start 97.505737 138.224237) (end 96.9495 137.668) (width 0.254) (layer B.Cu) (net 5))
   (segment (start 119.528949 143.675013) (end 102.956513 143.675013) (width 0.254) (layer B.Cu) (net 5))
@@
   (segment (start 274.79625 116.74475) (end 273.332599 118.208401) (width 0.254) (layer B.Cu) (net 54))
   (segment (start 274.79625 110.8075) (end 274.79625 116.74475) (width 0.254) (layer B.Cu) (net 54))
-  (segment (start 146.83125 74.5405) (end 146.83125 76.43475) (width 0.381) (layer B.Cu) (net 55))
-  (segment (start 146.83125 76.43475) (end 146.812 76.454) (width 0.381) (layer B.Cu) (net 55))
-  (segment (start 146.812 84.3885) (end 146.84375 84.42025) (width 0.381) (layer B.Cu) (net 55))
-  (segment (start 146.812 82.54575) (end 146.812 84.3885) (width 0.381) (layer B.Cu) (net 55))
-  (segment (start 146.83125 74.5405) (end 146.83125 69.778) (width 0.381) (layer B.Cu) (net 55))
-  (segment (start 146.812 76.454) (end 146.812 82.54575) (width 0.381) (layer B.Cu) (net 55))
+  (segment (start 146.84375 69.7905) (end 146.83125 69.778) (width 0.381) (layer B.Cu) (net 55))
+  (segment (start 146.84375 81.658) (end 146.84375 69.7905) (width 0.381) (layer B.Cu) (net 55))
   (segment (start 20.79625 91.91625) (end 23.1775 94.2975) (width 0.254) (layer F.Cu) (net 56))
   (segment (start 20.79625 75.2475) (end 20.79625 91.91625) (width 0.254) (layer F.Cu) (net 56))
@@
   (segment (start 126.328 125.73) (end 123.888 128.17) (width 0.254) (layer B.Cu) (net 75))
   (segment (start 129.2375 125.73) (end 126.328 125.73) (width 0.254) (layer B.Cu) (net 75))
+  (zone (net 1) (net_name GND) (layer B.Cu) (hatch edge 0.508)
+    (connect_pads (clearance 0.508))
+    (min_thickness 0.254)
+    (fill yes (arc_segments 32) (thermal_gap 0.508) (thermal_bridge_width 0.508))
+    (polygon
+      (pts
+        (xy 156.36875 63.5) (xy 140.49375 63.5) (xy 140.49375 68.2625) (xy 15.08125 68.2625) (xy 15.08125 144.4625)
+        (xy 281.78125 144.4625) (xy 281.78125 68.2625) (xy 156.36875 68.2625)
+      )
+    )
+  )
 )
